File: hardware/eagle/MCU/motor_breakout.sch (EAGLE design)
At the start: 17 parts, among them X1 1751248, X2 1751248

Commit message: added ground pour and power connection to MCU breakout
Connections:
- removed net N$10: U$2.8
- net VDD: now also U$2.8
