File: hardware/eagle/Arduino board/baord1.sch (EAGLE design)
At the start: 144 parts, among them Q1 BSS138, Q2 BSS138, U1 ARDUINO-MEGAFULL, U2 WIZ811MJ, U3 LSM303DLHC, U4 RT9193, U5 PCA9685, X1 1751248, X10 1751248, X11 1751248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

Commit message: All components added to PCB schematic: Arduino, ethernet, 6 MCUs, GPIO expander, PWM expander
Parts:
- added U$63: TCA6424A, netpune:TCA6424A
Connections:
- removed net BRK@1: R5.1, U$1.MODE1, U$2.1
- removed net BRK@2: R13.1, U$3.MODE1, U$4.1
- removed net BRK@3: R21.1, U$17.MODE1, U$18.1
- removed net BRK@4: R29.1, U$19.MODE1, U$20.1
- removed net BRK@5: R37.1, U$21.MODE1, U$22.1
- removed net BRK@6: R45.1, U$23.MODE1, U$24.1
- removed net CS@1: C10.1, R11.2, U$2.4
- removed net CS@2: C15.1, C37.1, R19.2, U$4.4
- removed net CS@3: C20.1, R27.2, U$18.4
- removed net CS@4: C25.1, R35.2, U$20.4
- removed net CS@5: C30.1, R43.2, U$22.4
- removed net CS@6: C35.1, R51.2, U$24.4
- removed net DIR@1: U$1.PHASE, U$2.5
- removed net DIR@2: U$3.PHASE, U$4.5
- removed net DIR@3: U$17.PHASE, U$18.5
- removed net DIR@4: U$19.PHASE, U$20.5
- removed net DIR@5: U$21.PHASE, U$22.5
- removed net DIR@6: U$23.PHASE, U$24.5
- removed net FLT@1: R9.1, U$1.FAULT, U$2.2
- removed net FLT@2: R17.1, U$3.FAULT, U$4.2
- removed net FLT@3: R25.1, U$17.FAULT, U$18.2
- removed net FLT@4: R33.1, U$19.FAULT, U$20.2
- removed net FLT@5: R41.1, U$21.FAULT, U$22.2
- removed net FLT@6: R49.1, U$23.FAULT, U$24.2
- removed net PWM@1: R7.2, U$1.ENABLE, U$2.7, U5.PWM1
- removed net PWM@2: R15.2, U$3.ENABLE, U$4.7, U5.PWM2
- removed net PWM@3: R23.2, U$17.ENABLE, U$18.7, U5.PWM3
- removed net PWM@4: R31.2, U$19.ENABLE, U$20.7, U5.PWM4
- removed net PWM@5: R39.2, U$21.ENABLE, U$22.7, U5.PWM5
- removed net PWM@6: R47.2, U$23.ENABLE, U$24.7, U5.PWM6
- removed net SLP@1: R6.1, U$1.SLEEP, U$2.3
- removed net SLP@2: R14.1, U$3.SLEEP, U$4.3
- removed net SLP@3: R22.1, U$17.SLEEP, U$18.3
- removed net SLP@4: R30.1, U$19.SLEEP, U$20.3
- removed net SLP@5: R38.1, U$21.SLEEP, U$22.3
- removed net SLP@6: R46.1, U$23.SLEEP, U$24.3
- new net BRK1: R5.1, U$1.MODE1, U$2.1, U$63.P00
- new net BRK2: R13.1, U$3.MODE1, U$4.1, U$63.P04
- new net BRK3: R21.1, U$17.MODE1, U$18.1, U$63.P10
- new net BRK4: R29.1, U$19.MODE1, U$20.1, U$63.P14
- new net BRK5: R37.1, U$21.MODE1, U$22.1, U$63.P20
- new net BRK6: R45.1, U$23.MODE1, U$24.1, U$63.P24
- new net CS1: C10.1, R11.2, U$2.4, U1.A10
- new net CS2: C15.1, C37.1, R19.2, U$4.4, U1.A11
- new net CS3: C20.1, R27.2, U$18.4, U1.A12
- new net CS4: C25.1, R35.2, U$20.4, U1.A13
- new net CS5: C30.1, R43.2, U$22.4, U1.A14
- new net CS6: C35.1, R51.2, U$24.4, U1.A15
- new net DIR1: U$1.PHASE, U$2.5, U$63.P02
- new net DIR2: U$3.PHASE, U$4.5, U$63.P06
- new net DIR3: U$17.PHASE, U$18.5, U$63.P12
- new net DIR4: U$19.PHASE, U$20.5, U$63.P16
- new net DIR5: U$21.PHASE, U$22.5, U$63.P22
- new net DIR6: U$23.PHASE, U$24.5, U$63.P26
- new net FLT1: R9.1, U$1.FAULT, U$2.2, U$63.P03
- new net FLT2: R17.1, U$3.FAULT, U$4.2, U$63.P07
- new net FLT3: R25.1, U$17.FAULT, U$18.2, U$63.P13
- new net FLT4: R33.1, U$19.FAULT, U$20.2, U$63.P17
- new net FLT5: R41.1, U$21.FAULT, U$22.2, U$63.P23
- new net FLT6: R49.1, U$23.FAULT, U$24.2, U$63.P27
- new net GPIO_INT: U$63.INT, U1.38
- new net GPIO_RES: U$63.RESET, U1.39
- new net SLP1: R6.1, U$1.SLEEP, U$2.3, U$63.P01
- new net SLP2: R14.1, U$3.SLEEP, U$4.3, U$63.P05
- new net SLP3: R22.1, U$17.SLEEP, U$18.3, U$63.P11
- new net SLP4: R30.1, U$19.SLEEP, U$20.3, U$63.P15
- new net SLP5: R38.1, U$21.SLEEP, U$22.3, U$63.P21
- new net SLP6: R46.1, U$23.SLEEP, U$24.3, U$63.P25
- net GND: now also U$63.ADDR, U$63.GND, U1.GND@0, U1.GND@1, U1.GND@2, U1.GND@3, U1.GND@4
- net PWM1: now also R7.2, U$1.ENABLE, U$2.7, U5.PWM1
- net PWM2: now also R15.2, U$3.ENABLE, U$4.7, U5.PWM2
- net PWM3: now also R23.2, U$17.ENABLE, U$18.7, U5.PWM3
- net PWM4: now also R31.2, U$19.ENABLE, U$20.7, U5.PWM4
- net PWM5: now also R39.2, U$21.ENABLE, U$22.7, U5.PWM5
- net PWM6: now also R47.2, U$23.ENABLE, U$24.7, U5.PWM6
- net SCL_5V: now also U$63.SCL, U1.21(SCL)
- net SDA_5V: now also U$63.SDA, U1.20(SDA)
- net VDD: now also U$63.VCCP, U1.5V@0, U1.5V@1, U1.5V@2, U1.VIN
