File: hw/output.sch (EAGLE design)
At the start: 22 parts, among them Q1 MOSFET-NCHANNELFDD8780, Q2 MOSFET-NCHANNELFDD8780, U3 TMP102

Commit message: Consolidated output board to use single control IC (CY8C9540A), removed servo pwm lines for this revision.
Parts:
- removed R3: 1K, SparkFun-Resistors:1KOHM-1/10W-1%(0603)
- removed U2: (no value), SparkFun-DigitalIC:SX1509
- U$5: value PCF8575C -> CY8C9540A; device SparkFun-DigitalIC:PCF8575C -> SpaceY:CY8C9540A
Connections:
- removed net N$1: U$5.INT
- removed net N$42: U2.OSCIO
- removed net N$43: U2.!INT
- net AIN1: no longer U$5.PO0
- net AIN2: no longer U$5.PO1
- net B1: now also X1.4; no longer X1.3
- net B2: now also X1.3; no longer X1.4
- net BIN1: no longer U$5.PO2
- net BIN2: no longer U$5.PO3
- net CIN1: no longer U$5.PO4
- net CIN2: no longer U$5.PO5
- net D1: now also X1.8; no longer X1.7
- net D2: now also X1.7; no longer X1.8
- net DIN1: no longer U$5.PO6
- net DIN2: no longer U$5.PO7
- net EIN1: no longer U$5.P10
- net EIN2: no longer U$5.P11
- net F1: now also X1.12; no longer X1.11
- net F2: now also X1.11; no longer X1.12
- net FIN1: no longer U$5.P12
- net FIN2: no longer U$5.P13
- net GIN1: no longer U$5.P14
- net GIN2: no longer U$5.P15
- net GND: now also U$5.GND@1, U$5.GND@2, U$5.INT; no longer U$5.A0, U$5.A1, U$5.A2, U$5.GND, U2.GND
- net H1: now also X1.25; no longer X1.24
- net H2: now also X1.24; no longer X1.25
- net HIN1: no longer U$5.P16
- net HIN2: no longer U$5.P17
- net LED1: now also U$5.P1_B4; no longer U2.I/O[9]
- net LED2: now also U$5.P1_B5; no longer U2.I/O[10]
- net PWM_A: now also U$5.P1_B0; no longer U2.I/O[0]
- net PWM_B: now also U$5.P0_B0; no longer U2.I/O[1]
- net PWM_C: now also U$5.P1_B1; no longer U2.I/O[2]
- net PWM_D: now also U$5.P0_B1; no longer U2.I/O[3]
- net PWM_E: now also U$5.P1_B2; no longer U2.I/O[4]
- net PWM_F: now also U$5.P0_B2; no longer U2.I/O[5]
- net PWM_G: now also U$5.P1_B3; no longer U2.I/O[6]
- net PWM_H: now also U$5.P0_B3; no longer U2.I/O[7]
- net RESET: no longer R3.1, U2.!RESET
- net SCL: no longer U2.SCL
- net SDA: no longer U2.SDA
- net SERVO1: no longer U2.I/O[11]
- net SERVO2: no longer U2.I/O[12]
- net SERVO3: no longer U2.I/O[13]
- net SERVO4: no longer U2.I/O[14]
- net SERVO5: no longer U2.I/O[15]
- net STBY: no longer U2.I/O[8]
- net VCC: now also U$5.A0; no longer R3.2, U2.ADDR0, U2.ADDR1, U2.VCC1, U2.VCC2, U2.VDDM
Other:
- note added: "5V Regulator"
