File: hw/Output/output.sch (EAGLE design)
At the start: 20 parts, among them Q1 MOSFET-NCHANNELFDD8780, Q2 MOSFET-NCHANNELFDD8780, U3 TMP102

Commit message: Added power indication LED and Battery current/voltage measurement to output board. Added atmega32u2, IMU header, Temp sensor connector, and wiz55io header to control board.
Parts:
- added C5, C6, C7: 0.1uF, SparkFun-Capacitors:0.1UF-25V-5%(0603)
- added LED1: (no value), SparkFun-LED:LED0603
- added R3: .1/1%, SparkFun-Passives:RESISTOR2512
- added R6: (no value), SparkFun-Passives:RESISTOR0603-RES
- added U$6: INA219, INA219:INA219
Connections:
- new net N$1: LED1.A, R6.1
- new net V_BATT_IN: R3.1, U$6.VIN+, X1.21
- net GND: now also C5.2, C6.2, C7.2, LED1.C, U$6.A0, U$6.A1, U$6.GND
- net SCL: now also U$6.SCL
- net SDA: now also U$6.SDA
- net VCC: now also C5.1, C6.1, U$6.VS
- net V_BATT: now also C7.1, R3.2, R6.2, U$6.VIN-; no longer X1.21
Changed lines of the file:
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@@
 <part name="GND20" library="SparkFun-Aesthetics" deviceset="GND" device=""/>
 <part name="U$5" library="SpaceY" deviceset="CY8C9540A" device=""/>
+<part name="U$6" library="INA219" deviceset="INA219" device=""/>
+<part name="GND11" library="SparkFun-Aesthetics" deviceset="GND" device=""/>
+<part name="SUPPLY15" library="SparkFun-Aesthetics" deviceset="VCC" device=""/>
+<part name="GND17" library="SparkFun-Aesthetics" deviceset="GND" device=""/>
+<part name="C5" library="SparkFun-Capacitors" deviceset="0.1UF-25V-5%(0603)" device="" value="0.1uF"/>
+<part name="C6" library="SparkFun-Capacitors" deviceset="0.1UF-25V-5%(0603)" device="" value="0.1uF"/>
+<part name="R3" library="SparkFun-Passives" deviceset="RESISTOR" device="2512" value=".1/1%"/>
+<part name="C7" library="SparkFun-Capacitors" deviceset="0.1UF-25V-5%(0603)" device="" value="0.1uF"/>
+<part name="R6" library="SparkFun-Passives" deviceset="RESISTOR" device="0603-RES"/>
+<part name="LED1" library="SparkFun-LED" deviceset="LED" device="0603"/>
+<part name="GND21" library="SparkFun-Aesthetics" deviceset="GND" device=""/>
+<part name="SUPPLY17" library="SparkFun-Aesthetics" deviceset="V_BATT" device=""/>
 </parts>
 <sheets>
@@
 <instance part="GND20" gate="1" x="134.62" y="-88.9"/>
 <instance part="U$5" gate="G$1" x="248.92" y="132.08"/>
+<instance part="U$6" gate="G$1" x="-55.88" y="144.78" rot="R90"/>
+<instance part="GND11" gate="1" x="-30.48" y="149.86"/>
+<instance part="SUPPLY15" gate="G$1" x="-91.44" y="142.24"/>
+<instance part="GND17" gate="1" x="-73.66" y="129.54"/>
+<instance part="C5" gate="G$1" x="17.78" y="182.88"/>
+<instance part="C6" gate="G$1" x="-86.36" y="137.16"/>
+<instance part="R3" gate="G$1" x="-20.32" y="139.7" rot="R90"/>
+<instance part="C7" gate="G$1" x="-7.62" y="182.88"/>
+<instance part="R6" gate="G$1" x="-30.48" y="172.72" rot="R180"/>
+<instance part="LED1" gate="G$1" x="-17.78" y="172.72" rot="R90"/>
+<instance part="GND21" gate="1" x="-5.08" y="170.18"/>
+<instance part="SUPPLY17" gate="G$1" x="-38.1" y="172.72"/>
 </instances>
 <busses>
@@
 <wire x1="5.08" y1="180.34" x2="5.08" y2="175.26" width="0.1524" layer="91"/>
 <pinref part="GND14" gate="1" pin="GND"/>
+<pinref part="C7" gate="G$1" pin="2"/>
+<wire x1="-7.62" y1="180.34" x2="5.08" y2="180.34" width="0.1524" layer="91"/>
+<junction x="5.08" y="180.34"/>
+<pinref part="C5" gate="G$1" pin="2"/>
+<wire x1="17.78" y1="180.34" x2="5.08" y2="180.34" width="0.1524" layer="91"/>
 </segment>
 <segment>
@@
 <wire x1="266.7" y1="73.66" x2="266.7" y2="88.9" width="0.1524" layer="91"/>
 </segment>
+<segment>
+<pinref part="U$6" gate="G$1" pin="GND"/>
+<wire x1="-73.66" y1="137.16" x2="-73.66" y2="134.62" width="0.1524" layer="91"/>
+<pinref part="GND17" gate="1" pin="GND"/>
+<pinref part="C6" gate="G$1" pin="2"/>
+<wire x1="-73.66" y1="134.62" x2="-73.66" y2="132.08" width="0.1524" layer="91"/>
+<wire x1="-86.36" y1="134.62" x2="-73.66" y2="134.62" width="0.1524" layer="91"/>
+<junction x="-73.66" y="134.62"/>
+</segment>
+<segment>
+<pinref part="U$6" gate="G$1" pin="A1"/>
+<wire x1="-40.64" y1="152.4" x2="-35.56" y2="152.4" width="0.1524" layer="91"/>
+<pinref part="GND11" gate="1" pin="GND"/>
+<pinref part="U$6" gate="G$1" pin="A0"/>
+<wire x1="-35.56" y1="152.4" x2="-30.48" y2="152.4" width="0.1524" layer="91"/>
+<wire x1="-40.64" y1="147.32" x2="-35.56" y2="147.32" width="0.1524" layer="91"/>
+<wire x1="-35.56" y1="147.32" x2="-35.56" y2="152.4" width="0.1524" layer="91"/>
+<junction x="-35.56" y="152.4"/>
+</segment>
+<segment>
+<pinref part="LED1" gate="G$1" pin="C"/>
+<wire x1="-12.7" y1="172.72" x2="-5.08" y2="172.72" width="0.1524" layer="91"/>
+<pinref part="GND21" gate="1" pin="GND"/>
+</segment>
 </net>
 <net name="SERVO1" class="0">
@@
 <wire x1="276.86" y1="88.9" x2="276.86" y2="78.74" width="0.1524" layer="91"/>
 </segment>
+<segment>
+<pinref part="U$6" gate="G$1" pin="SDA"/>
+<wire x1="-73.66" y1="152.4" x2="-83.82" y2="152.4" width="0.1524" layer="91"/>
+<label x="-83.82" y="152.4" size="1.778" layer="95"/>
+</segment>
 </net>
 <net name="SCL" class="0">
@@
 <pinref part="U$5" gate="G$1" pin="SCL"/>
 <wire x1="271.78" y1="88.9" x2="271.78" y2="78.74" width="0.1524" layer="91"/>
+</segment>
+<segment>
+<pinref part="U$6" gate="G$1" pin="SCL"/>
+<wire x1="-73.66" y1="147.32" x2="-83.82" y2="147.32" width="0.1524" layer="91"/>
+<label x="-83.82" y="147.32" size="1.778" layer="95"/>
 </segment>
 </net>
@@
 <segment>
 <pinref part="IC1" gate="G$1" pin="IN"/>
-<wire x1="-2.54" y1="187.96" x2="-12.7" y2="187.96" width="0.1524" layer="91"/>
+<wire x1="-2.54" y1="187.96" x2="-7.62" y2="187.96" width="0.1524" layer="91"/>
 <pinref part="SUPPLY21" gate="G$1" pin="V_BATT"/>
-</segment>
-<segment>
-<pinref part="X1" gate="-1" pin="21"/>
-<wire x1="-53.34" y1="58.42" x2="-48.26" y2="58.42" width="0.1524" layer="91"/>
-<label x="-53.34" y="58.42" size="1.778" layer="95"/>
+<pinref part="C7" gate="G$1" pin="1"/>
+<wire x1="-7.62" y1="187.96" x2="-12.7" y2="187.96" width="0.1524" layer="91"/>
+<junction x="-7.62" y="187.96"/>
+</segment>
+<segment>
+<pinref part="U$6" gate="G$1" pin="VIN-"/>
+<wire x1="-40.64" y1="142.24" x2="-25.4" y2="142.24" width="0.1524" layer="91"/>
+<label x="-38.1" y="142.24" size="1.778" layer="95"/>
+<pinref part="R3" gate="G$1" pin="2"/>
+<wire x1="-25.4" y1="142.24" x2="-20.32" y2="144.78" width="0.1524" layer="91"/>
+</segment>
+<segment>
+<pinref part="R6" gate="G$1" pin="2"/>
+<pinref part="SUPPLY17" gate="G$1" pin="V_BATT"/>
+<wire x1="-38.1" y1="172.72" x2="-35.56" y2="172.72" width="0.1524" layer="91"/>
 </segment>
 </net>
@@
 <segment>
 <pinref part="IC1" gate="G$1" pin="OUT"/>
-<wire x1="12.7" y1="187.96" x2="22.86" y2="187.96" width="0.1524" layer="91"/>
+<wire x1="12.7" y1="187.96" x2="17.78" y2="187.96" width="0.1524" layer="91"/>
 <pinref part="SUPPLY22" gate="G$1" pin="VCC"/>
+<pinref part="C5" gate="G$1" pin="1"/>
+<wire x1="17.78" y1="187.96" x2="22.86" y2="187.96" width="0.1524" layer="91"/>
+<junction x="17.78" y="187.96"/>
 </segment>
 <segment>
@@
 <wire x1="261.62" y1="88.9" x2="261.62" y2="71.12" width="0.1524" layer="91"/>
 </segment>
+<segment>
+<pinref part="U$6" gate="G$1" pin="VS"/>
+<pinref part="SUPPLY15" gate="G$1" pin="VCC"/>
+<wire x1="-73.66" y1="142.24" x2="-86.36" y2="142.24" width="0.1524" layer="91"/>
+<pinref part="C6" gate="G$1" pin="1"/>
+<wire x1="-86.36" y1="142.24" x2="-91.44" y2="142.24" width="0.1524" layer="91"/>
+<junction x="-86.36" y="142.24"/>
+</segment>
 </net>
 <net name="LEDIN1" class="0">
@@
 </segment>
 </net>
+<net name="V_BATT_IN" class="0">
+<segment>
+<pinref part="U$6" gate="G$1" pin="VIN+"/>
+<wire x1="-40.64" y1="137.16" x2="-25.4" y2="137.16" width="0.1524" layer="91"/>
+<label x="-38.1" y="137.16" size="1.778" layer="95"/>
+<pinref part="R3" gate="G$1" pin="1"/>
+<wire x1="-25.4" y1="137.16" x2="-20.32" y2="134.62" width="0.1524" layer="91"/>
+</segment>
+<segment>
+<pinref part="X1" gate="-1" pin="21"/>
+<wire x1="-53.34" y1="58.42" x2="-48.26" y2="58.42" width="0.1524" layer="91"/>
+<label x="-53.34" y="58.42" size="1.778" layer="95"/>
+</segment>
+</net>
+<net name="N$1" class="0">
+<segment>
+<pinref part="R6" gate="G$1" pin="1"/>
+<pinref part="LED1" gate="G$1" pin="A"/>
+<wire x1="-20.32" y1="172.72" x2="-25.4" y2="172.72" width="0.1524" layer="91"/>
+</segment>
+</net>

Commit message: Added Power Switch to output board.
Parts:
- added S1: (no value), SparkFun-Electromechanical:SWITCH-SPDTKIT
Connections:
- new net BATT: S1.P, X1.21
- net V_BATT_IN: now also S1.S; no longer X1.21
Changed lines of the file:
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@@
 <part name="GND21" library="SparkFun-Aesthetics" deviceset="GND" device=""/>
 <part name="SUPPLY17" library="SparkFun-Aesthetics" deviceset="V_BATT" device=""/>
+<part name="S1" library="SparkFun-Electromechanical" deviceset="SWITCH-SPDT" device="KIT"/>
 </parts>
 <sheets>
@@
 <instance part="GND21" gate="1" x="-5.08" y="170.18"/>
 <instance part="SUPPLY17" gate="G$1" x="-38.1" y="172.72"/>
+<instance part="S1" gate="1" x="-45.72" y="91.44"/>
 </instances>
 <busses>
@@
 </segment>
 <segment>
+<pinref part="S1" gate="1" pin="S"/>
+<wire x1="-40.64" y1="88.9" x2="-33.02" y2="88.9" width="0.1524" layer="91"/>
+<label x="-35.56" y="88.9" size="1.778" layer="95"/>
+</segment>
+</net>
+<net name="N$1" class="0">
+<segment>
+<pinref part="R6" gate="G$1" pin="1"/>
+<pinref part="LED1" gate="G$1" pin="A"/>
+<wire x1="-20.32" y1="172.72" x2="-25.4" y2="172.72" width="0.1524" layer="91"/>
+</segment>
+</net>
+<net name="BATT" class="0">
+<segment>
+<pinref part="S1" gate="1" pin="P"/>
+<wire x1="-48.26" y1="91.44" x2="-55.88" y2="91.44" width="0.1524" layer="91"/>
+<label x="-55.88" y="91.44" size="1.778" layer="95"/>
+</segment>
+<segment>
 <pinref part="X1" gate="-1" pin="21"/>
 <wire x1="-53.34" y1="58.42" x2="-48.26" y2="58.42" width="0.1524" layer="91"/>
@@
 </segment>
 </net>
-<net name="N$1" class="0">
-<segment>
-<pinref part="R6" gate="G$1" pin="1"/>
-<pinref part="LED1" gate="G$1" pin="A"/>
-<wire x1="-20.32" y1="172.72" x2="-25.4" y2="172.72" width="0.1524" layer="91"/>
-</segment>
-</net>
